File: hardware/radiationsensor_r1/arrayboard_r0.sch (EAGLE design)
At the start: 21 parts, among them CN0 RADIATION-SENSOR-REV1, CN1 RADIATION-SENSOR-REV1, CN10 RADIATION-SENSOR-REV1, CN11 RADIATION-SENSOR-REV1, CN12 RADIATION-SENSOR-REV1, CN13 RADIATION-SENSOR-REV1, CN14 RADIATION-SENSOR-REV1, CN15 RADIATION-SENSOR-REV1, CN16 2524-, CN17 22-23-2041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

Commit message: Added MCU to Array board
Parts:
- removed CN16: 2524-, con-3m:2524-
- added AT32U4: ATMEGA32U4TQFP-44, SparkFun-DigitalIC:ATMEGA32U4TQFP-44
- added C2: 100nF, SparkFun-Passives:CAP0805
- added C3: 1uF, SparkFun-Passives:CAP0805
- added JP1: AVR_SPI_PRG_6PTH, SparkFun-Connectors:AVR_SPI_PRG_6PTH
- added JP2: USB-MICROB, SparkFun-Connectors:USB-MICROB
- added JP3: (no value), SparkFun-Connectors:M04POLAR
- added R2, R3: 22, SparkFun-Passives:RESISTOR0805-RES
- added R4: 10K, SparkFun-Passives:RESISTOR0805-RES
- added Y1: 16MHZ, SparkFun-FreqCtrl:RESONATOR16MHZ
Connections:
- removed net COMP1: CN1.COMP_OUT, CN16-2.KL
- new net MISO/COMP1: AT32U4.PB3(MISO), CN1.COMP_OUT, JP1.1
- new net N$1: JP2.D-, R3.1
- new net N$3: JP2.D+, R2.1
- new net N$4: AT32U4.UCAP, C3.2
- new net N$5: AT32U4.XTAL1, Y1.1
- new net N$6: AT32U4.UVCC
- new net N$7: AT32U4.XTAL2, Y1.3
- new net N$9: AT32U4.AREF, C2.2
- new net RST: AT32U4.!RESET, JP1.5, R4.1
- new net RX: AT32U4.PD2(RX), JP3.2
- new net TX: AT32U4.PD3(TX), JP3.3
- new net USB+: AT32U4.D+, R3.2
- new net USB-: AT32U4.D-, R2.2
- net COMP0: now also AT32U4.PE6; no longer CN16-1.KL
- net COMP10: now also AT32U4.PC6; no longer CN16-11.KL
- net COMP11: now also AT32U4.PC7; no longer CN16-12.KL
- net COMP12: now also AT32U4.PF7(ADC7); no longer CN16-13.KL
- net COMP13: now also AT32U4.PF6(ADC6); no longer CN16-14.KL
- net COMP14: now also AT32U4.PF5(ADC5); no longer CN16-15.KL
- net COMP15: now also AT32U4.PF4(ADC4); no longer CN16-16.KL
- net COMP2: now also AT32U4.PB7; no longer CN16-3.KL
- net COMP3: now also AT32U4.PD5; no longer CN16-4.KL
- net COMP4: now also AT32U4.PD4(ADC8); no longer CN16-5.KL
- net COMP5: now also AT32U4.PD6(ADC9); no longer CN16-6.KL
- net COMP6: now also AT32U4.PD7(ADC10); no longer CN16-7.KL
- net COMP7: now also AT32U4.PB4(ADC11); no longer CN16-8.KL
- net COMP8: now also AT32U4.PB5(ADC12); no longer CN16-9.KL
- net COMP9: now also AT32U4.PB6(ADC13); no longer CN16-10.KL
- net GND: now also AT32U4.GND@15, AT32U4.GND@23, AT32U4.GND@35, AT32U4.GND@43, AT32U4.UGND, C2.1, C3.1, JP1.6, JP2.GND, JP3.4, Y1.2; no longer CN16-24.KL
- net MOSI: now also AT32U4.PB2(MOSI), JP1.4; no longer CN16-20.KL
- net SCL: now also AT32U4.PD0(SCL); no longer CN16-17.KL
- net SCLK: now also AT32U4.PB1(SCK), JP1.3; no longer CN16-19.KL
- net SDA: now also AT32U4.PD1(SDA); no longer CN16-18.KL
- net VLOGIC: now also AT32U4.AVCC@24, AT32U4.AVCC@44, AT32U4.VBUS, AT32U4.VCC@14, AT32U4.VCC@34, JP1.2, JP2.VBUS, JP3.1, R4.2; no longer CN16-23.KL
- net VTEMP11: now also AT32U4.PF0(ADC0); no longer CN16-22.KL
- net VTEMP4: now also AT32U4.PF1(ADC1); no longer CN16-21.KL
Other:
- note added: "ICSP INTERFACE"
- note added: "MICROCONTROLLER"
- note added: "SERIAL INTERFACE"
- note added: "USB INTERFACE"
- note removed: "MICROCONTROLLER CONNECTOR"
- moved on the sheet: CN17-1, CN17-2, CN17-3, CN17-4
